File: 1802-Mini-Serial-1854.kicad_pcb (KiCad board)
At the start: 2 copper layers, 100 x 100 mm, 46 parts, among them J1 Mount, J10 TTL, J2 Mount, J3 Mount, J4 Mount, J5 Expansion, J6 GRP_EXP, J7 GRP_SEL, J8 DCE, J9 DTE, U1 4001, U10 4051, U11 MAX232, U2 CDP1854, U3 4049, U4 4071, U5 4023, U6 4013, U7 74LS174, U8 4024, U9 4019, X1 1.8432

Commit message: Fix EF flags
Connections:
- JP3 pad 1: ~EF2 -> ~EF3
- JP4 pad 3: ~EF3 -> ~EF2
Routing:
- net ~EF2: track 26.6 -> 14.7 mm
- net ~EF3: track 15.9 -> 15.0 mm
- net ~EF4: track 11.4 -> 12.0 mm

Commit message: Layout fixes
Parts:
- renumbered C6 to C1, C1 to C2, C5 to C3, C2 to C4, C4 to C5, C7 to C6, C9 to C7, D2 to D1, D1 to D2, U2 to U1, U8 to U10, U6 to U11, U3 to U2, U7 to U3, U9 to U4, U10 to U5, U11 to U6, U4 to U7, U5 to U8, U1 to U9
Routing:
- net GND: track 10.6 -> 13.1 mm, vias 1 -> 3
- net VCC: track 390.3 -> 388.1 mm
- net ~MRD: track 118.5 -> 120.1 mm
- net (no net): vias 2 -> 0

Commit message: Add files via upload
Routing:
- net GND: vias 3 -> 1
Changed lines of the file:
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@@
     (thickness 1.6)
     (drawings 450)
-    (tracks 1004)
+    (tracks 1002)
     (zones 0)
     (modules 46)
@@
   (segment (start 157.48 146.05) (end 157.48 144.145) (width 0.750013) (layer B.Cu) (net 1))
   (segment (start 157.48 146.05) (end 157.48 143.51) (width 0.750013) (layer F.Cu) (net 1))
-  (via (at 106.045 136.2075) (size 0.6) (drill 0.4) (layers F.Cu B.Cu) (net 1))
   (segment (start 157.48 146.05) (end 157.48 143.51) (width 0.750013) (layer B.Cu) (net 1))
-  (via (at 118.745 137.16) (size 0.6) (drill 0.4) (layers F.Cu B.Cu) (net 1))
   (via (at 164.465 132.715) (size 0.6) (drill 0.4) (layers F.Cu B.Cu) (net 1))
   (segment (start 154.94 145.415) (end 154.94 146.05) (width 0.25) (layer F.Cu) (net 2) (status 30))
